File: projects/Z-LiDAR_Demo_Board-VL53L0X-TM4C123GXL/LiDAR_Demo_Board.brd (EAGLE design)
At the start: 91.4 x 89.8 mm, 9 parts, among them IC1 EK-TM4C123GXLP

Commit message: fixed some tiny inperfections
Changed lines of the file:
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@@
 <element name="IC1" library="UT_ECE" package="TM4C123LAUNCHPAD" value="EK-TM4C123GXLP" x="132.715" y="44.45" smashed="yes" rot="R180">
 <attribute name="NAME" x="150.749" y="27.051" size="1.778" layer="25" font="vector" ratio="10"/>
-<attribute name="VALUE" x="114.935" y="28.9052" size="1.778" layer="25" font="vector" ratio="10" rot="R180"/>
 </element>
 <element name="U$1" library="Z" package="VL53L0X_ATK" value="VL53L0X_ATK" x="71.12" y="71.12" smashed="yes"/>
